File: thermostat/misc.kicad_sch (KiCad schematic)
At the start: 8 parts

Commit message: layout with holes to fit in old slot
Parts:
- H1: footprint MountingHole:MountingHole_2.2mm_M2_DIN965_Pad_TopBottom -> kelvie:MountingHole_No6_Pad_TopBottom
- H2: footprint (none) -> kelvie:MountingHole_No6_Pad_TopBottom
- H3, H4, H5, H6, H7, H8: footprint (none) -> MountingHole:MountingHole_2.2mm_M2_DIN965_Pad_TopBottom
Changed lines of the file:
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@@
       (effects (font (size 1.27 1.27)) (justify left))
     )
-    (property "Footprint" "" (id 2) (at 76.2 72.39 0)
+    (property "Footprint" "MountingHole:MountingHole_2.2mm_M2_DIN965_Pad_TopBottom" (id 2) (at 76.2 72.39 0)
       (effects (font (size 1.27 1.27)) hide)
     )
@@
       (effects (font (size 1.27 1.27)) (justify left))
     )
-    (property "Footprint" "" (id 2) (at 50.8 72.39 0)
+    (property "Footprint" "MountingHole:MountingHole_2.2mm_M2_DIN965_Pad_TopBottom" (id 2) (at 50.8 72.39 0)
       (effects (font (size 1.27 1.27)) hide)
     )
@@
       (effects (font (size 1.27 1.27)) (justify left))
     )
-    (property "Footprint" "MountingHole:MountingHole_2.2mm_M2_DIN965_Pad_TopBottom" (id 2) (at 34.29 72.39 0)
+    (property "Footprint" "kelvie:MountingHole_No6_Pad_TopBottom" (id 2) (at 34.29 72.39 0)
       (effects (font (size 1.27 1.27)) hide)
     )
@@
       (effects (font (size 1.27 1.27)) (justify left))
     )
-    (property "Footprint" "" (id 2) (at 64.77 72.39 0)
+    (property "Footprint" "MountingHole:MountingHole_2.2mm_M2_DIN965_Pad_TopBottom" (id 2) (at 64.77 72.39 0)
       (effects (font (size 1.27 1.27)) hide)
     )
@@
       (effects (font (size 1.27 1.27)) (justify left))
     )
-    (property "Footprint" "" (id 2) (at 43.18 72.39 0)
+    (property "Footprint" "kelvie:MountingHole_No6_Pad_TopBottom" (id 2) (at 43.18 72.39 0)
       (effects (font (size 1.27 1.27)) hide)
     )
@@
       (effects (font (size 1.27 1.27)) (justify left))
     )
-    (property "Footprint" "" (id 2) (at 71.12 72.39 0)
+    (property "Footprint" "MountingHole:MountingHole_2.2mm_M2_DIN965_Pad_TopBottom" (id 2) (at 71.12 72.39 0)
       (effects (font (size 1.27 1.27)) hide)
     )
@@
       (effects (font (size 1.27 1.27)) (justify left))
     )
-    (property "Footprint" "" (id 2) (at 81.28 72.39 0)
+    (property "Footprint" "MountingHole:MountingHole_2.2mm_M2_DIN965_Pad_TopBottom" (id 2) (at 81.28 72.39 0)
       (effects (font (size 1.27 1.27)) hide)
     )
@@
       (effects (font (size 1.27 1.27)) (justify left))
     )
-    (property "Footprint" "" (id 2) (at 57.15 72.39 0)
+    (property "Footprint" "MountingHole:MountingHole_2.2mm_M2_DIN965_Pad_TopBottom" (id 2) (at 57.15 72.39 0)
       (effects (font (size 1.27 1.27)) hide)
     )
